Commit message: SLAM works & ros2_control too

File: description/robot.urdf.xacro (robot description, xacro)
@@ -1,8 +1,12 @@
 <?xml version="1.0"?>
 <robot xmlns:xacro="http://www.ros.org/wiki/xacro"  name="robot">
+    <xacro:arg name="use_ros2_control" default="true"/>
     <xacro:include filename="robot_core.xacro" />
-<!--    <xacro:include filename="gazebo_control.xacro"/>
--->
-    <xacro:include filename="ros2_control.xacro" />
+    <xacro:if value="$(arg use_ros2_control)">
+        <xacro:include filename="ros2_control.xacro" />
+    </xacro:if>
+    <xacro:unless value="$(arg use_ros2_control)">
+        <xacro:include filename="gazebo_control.xacro" />
+    </xacro:unless>
     <xacro:include filename="lidar.xacro"/>
 <!--    <xacro:include filename="camera.xacro"/>        -->

File: description/robot_core.xacro (robot description, xacro)
@@ -20,5 +20,5 @@
     <link name="base_link">
     </link>
-    <!-- BASE FOOTPRINT LINK-->
+ <!-- BASE_FOOTPRINT LINK -->
     <joint name="base_footprint_joint" type="fixed">
         <parent link="base_link"/>
@@ -28,4 +28,5 @@
     <link name="base_footprint">
     </link>
+    <!--CHASSIS LINK-->
     <joint name="chassis_joint" type="fixed">
         <parent link="base_link"/>
@@ -71,5 +72,5 @@
         <collision>
             <geometry>
-                <cylinder radius="0.05" length="0.04"/>
+                <sphere radius="0.05"/>
             </geometry>
         </collision>
@@ -97,5 +98,5 @@
         <collision>
             <geometry>
-                <cylinder radius="0.05" length="0.04"/>
+                <sphere radius="0.05"/>
             </geometry>
         </collision>

File: install/wag_gsz_feleves/share/wag_gsz_feleves/description/robot.urdf.xacro (robot description, xacro)
@@ -1,6 +1,12 @@
 <?xml version="1.0"?>
 <robot xmlns:xacro="http://www.ros.org/wiki/xacro"  name="robot">
+    <xacro:arg name="use_ros2_control" default="true"/>
     <xacro:include filename="robot_core.xacro" />
-    <xacro:include filename="gazebo_control.xacro"/>
+    <xacro:if value="$(arg use_ros2_control)">
+        <xacro:include filename="ros2_control.xacro" />
+    </xacro:if>
+    <xacro:unless value="$(arg use_ros2_control)">
+        <xacro:include filename="gazebo_control.xacro" />
+    </xacro:unless>
     <xacro:include filename="lidar.xacro"/>
 <!--    <xacro:include filename="camera.xacro"/>        -->
